File: LongboardTailLights/LongboardTailLights.sch (KiCad schematic (older format))
At the start: 22 parts, among them P1 CONN_01X04, U1 AL8805, U2 AL8805

Commit message: small schematic changes
Parts:
- added JP2: JUMPER3, Connect:GS3, symbol JUMPER3
- added R5: 6200, Resistors_SMD:R_0603_HandSoldering, symbol R
- added R6: 1600, Resistors_SMD:R_0603_HandSoldering, symbol R
- C1, C5: footprint (none) -> Capacitors_SMD:C_0805_HandSoldering
- C2, C3, C4, C6, C7: footprint (none) -> Capacitors_SMD:C_0603_HandSoldering
- D3, D5: footprint (none) -> Light_Parts:PowerDI-123
- JP1: footprint (none) -> Connect:GS3
- L1, L2: footprint (none) -> Light_Parts:Inductor_Bourns_6045
- P1: footprint (none) -> Connectors_Molex:Molex_KK-6410-04_04x2.54mm_Straight
- R3: value R -> 6200
- R4: value R -> 1600
Connections:
- net CTRL1: now also JP2.2; no longer P1.4 (P4)
- net GND: now also R6.2
- net VCC: now also R5.1
- new net: JP2.1, R5.2, R6.1
- new net CTRL_EXT1: JP2.3, P1.4 (P4)
Changed lines of the file:
@@
 P 7550 3450
 F 0 "R4" V 7630 3450 50  0000 C CNN
-F 1 "R" V 7550 3450 50  0000 C CNN
+F 1 "1600" V 7550 3450 50  0000 C CNN
 F 2 "Resistors_SMD:R_0603_HandSoldering" V 7480 3450 50  0001 C CNN
 F 3 "" H 7550 3450 50  0000 C CNN
@@
 P 7550 3050
 F 0 "R3" V 7630 3050 50  0000 C CNN
-F 1 "R" V 7550 3050 50  0000 C CNN
+F 1 "6200" V 7550 3050 50  0000 C CNN
 F 2 "Resistors_SMD:R_0603_HandSoldering" V 7480 3050 50  0001 C CNN
 F 3 "" H 7550 3050 50  0000 C CNN
@@
 F 0 "C5" H 4575 3550 50  0000 L CNN
 F 1 "4.7uF" H 4575 3350 50  0000 L CNN
-F 2 "" H 4588 3300 50  0001 C CNN
+F 2 "Capacitors_SMD:C_0805_HandSoldering" H 4588 3300 50  0001 C CNN
 F 3 "" H 4550 3450 50  0000 C CNN
 	1    4550 3450
@@
 F 0 "C6" H 4825 3550 50  0000 L CNN
 F 1 "2.2uF" H 4825 3350 50  0000 L CNN
-F 2 "" H 4838 3300 50  0001 C CNN
+F 2 "Capacitors_SMD:C_0603_HandSoldering" H 4838 3300 50  0001 C CNN
 F 3 "" H 4800 3450 50  0000 C CNN
 	1    4800 3450
@@
 F 0 "C4" H 3575 4250 50  0000 L CNN
 F 1 "1uF" H 3575 4050 50  0000 L CNN
-F 2 "" H 3588 4000 50  0001 C CNN
+F 2 "Capacitors_SMD:C_0603_HandSoldering" H 3588 4000 50  0001 C CNN
 F 3 "" H 3550 4150 50  0000 C CNN
 	1    3550 4150
@@
 F 0 "C3" H 3575 3700 50  0000 L CNN
 F 1 "1uF" H 3575 3500 50  0000 L CNN
-F 2 "" H 3588 3450 50  0001 C CNN
+F 2 "Capacitors_SMD:C_0603_HandSoldering" H 3588 3450 50  0001 C CNN
 F 3 "" H 3550 3600 50  0000 C CNN
 	1    3550 3600
@@
 F 0 "C7" H 6425 3650 50  0000 L CNN
 F 1 "1uF" H 6425 3450 50  0000 L CNN
-F 2 "" H 6438 3400 50  0001 C CNN
+F 2 "Capacitors_SMD:C_0603_HandSoldering" H 6438 3400 50  0001 C CNN
 F 3 "" H 6400 3550 50  0000 C CNN
 	1    6400 3550
@@
 F 0 "L2" V 6100 4200 50  0000 C CNN
 F 1 "INDUCTOR" V 6250 4200 50  0000 C CNN
-F 2 "" H 6150 4200 50  0001 C CNN
+F 2 "Light_Parts:Inductor_Bourns_6045" H 6150 4200 50  0001 C CNN
 F 3 "" H 6150 4200 50  0000 C CNN
 	1    6150 4200
@@
 F 0 "L1" V 3250 4800 50  0000 C CNN
 F 1 "INDUCTOR" V 3400 4800 50  0000 C CNN
-F 2 "" H 3300 4800 50  0001 C CNN
+F 2 "Light_Parts:Inductor_Bourns_6045" H 3300 4800 50  0001 C CNN
 F 3 "" H 3300 4800 50  0000 C CNN
 	1    3300 4800
@@
 F 0 "D5" H 6700 3750 50  0000 C CNN
 F 1 "D_Schottky" H 6700 3550 50  0000 C CNN
-F 2 "" H 6700 3650 50  0001 C CNN
+F 2 "Light_Parts:PowerDI-123" H 6700 3650 50  0001 C CNN
 F 3 "" H 6700 3650 50  0000 C CNN
 	1    6700 3650
@@
 F 0 "D3" H 3850 3950 50  0000 C CNN
 F 1 "D_Schottky" H 3850 3750 50  0000 C CNN
-F 2 "" H 3850 3850 50  0001 C CNN
+F 2 "Light_Parts:PowerDI-123" H 3850 3850 50  0001 C CNN
 F 3 "" H 3850 3850 50  0000 C CNN
 	1    3850 3850
@@
 F 0 "C2" H 1975 3650 50  0000 L CNN
 F 1 "2.2uF" H 1975 3450 50  0000 L CNN
-F 2 "" H 1988 3400 50  0001 C CNN
+F 2 "Capacitors_SMD:C_0603_HandSoldering" H 1988 3400 50  0001 C CNN
 F 3 "" H 1950 3550 50  0000 C CNN
 	1    1950 3550
@@
 F 0 "C1" H 1725 3650 50  0000 L CNN
 F 1 "4.7uF" H 1725 3450 50  0000 L CNN
-F 2 "" H 1738 3400 50  0001 C CNN
+F 2 "Capacitors_SMD:C_0805_HandSoldering" H 1738 3400 50  0001 C CNN
 F 3 "" H 1700 3550 50  0000 C CNN
 	1    1700 3550
@@
 F 0 "JP1" H 8100 3150 50  0000 L CNN
 F 1 "JUMPER3" H 8050 3350 50  0000 C BNN
-F 2 "" H 8050 3250 50  0001 C CNN
+F 2 "Connect:GS3" H 8050 3250 50  0001 C CNN
 F 3 "" H 8050 3250 50  0000 C CNN
 	1    8050 3250
@@
 F 0 "P1" H 9200 3450 50  0000 C CNN
 F 1 "CONN_01X04" V 9300 3200 50  0000 C CNN
-F 2 "" H 9200 3200 50  0001 C CNN
+F 2 "Connectors_Molex:Molex_KK-6410-04_04x2.54mm_Straight" H 9200 3200 50  0001 C CNN
 F 3 "" H 9200 3200 50  0000 C CNN
 	1    9200 3200
@@
 $EndComp
 Text HLabel 9950 3050 2    60   Input ~ 0
+CTRL_EXT1
+Wire Wire Line
+	9950 3050 9400 3050
+$Comp
+L R R6
+U 1 1 57F46FD7
+P 7550 4800
+F 0 "R6" V 7630 4800 50  0000 C CNN
+F 1 "1600" V 7550 4800 50  0000 C CNN
+F 2 "Resistors_SMD:R_0603_HandSoldering" V 7480 4800 50  0001 C CNN
+F 3 "" H 7550 4800 50  0000 C CNN
+	1    7550 4800
+	1    0    0    -1
+$EndComp
+$Comp
+L R R5
+U 1 1 57F46FDD
+P 7550 4400
+F 0 "R5" V 7630 4400 50  0000 C CNN
+F 1 "6200" V 7550 4400 50  0000 C CNN
+F 2 "Resistors_SMD:R_0603_HandSoldering" V 7480 4400 50  0001 C CNN
+F 3 "" H 7550 4400 50  0000 C CNN
+	1    7550 4400
+	1    0    0    -1
+$EndComp
+Wire Wire Line
+	7550 4550 7550 4650
+Wire Wire Line
+	7550 4600 7800 4600
+Connection ~ 7550 4600
+$Comp
+L JUMPER3 JP2
+U 1 1 57F46FE6
+P 8050 4600
+F 0 "JP2" H 8100 4500 50  0000 L CNN
+F 1 "JUMPER3" H 8050 4700 50  0000 C BNN
+F 2 "Connect:GS3" H 8050 4600 50  0001 C CNN
+F 3 "" H 8050 4600 50  0000 C CNN
+	1    8050 4600
+	1    0    0    -1
+$EndComp
+Text HLabel 8000 5000 0    60   Input ~ 0
 CTRL1
 Wire Wire Line
-	9950 3050 9400 3050
+	8050 4700 8050 5000
+$Comp
+L GND #PWR011
+U 1 1 57F46FEE
+P 7550 5050
+F 0 "#PWR011" H 7550 4800 50  0001 C CNN
+F 1 "GND" H 7550 4900 50  0000 C CNN
+F 2 "" H 7550 5050 50  0000 C CNN
+F 3 "" H 7550 5050 50  0000 C CNN
+	1    7550 5050
+	1    0    0    -1
+$EndComp
+Wire Wire Line
+	7550 4950 7550 5050
+$Comp
+L VCC #PWR012
+U 1 1 57F46FF5
+P 7550 4150
+F 0 "#PWR012" H 7550 4000 50  0001 C CNN
+F 1 "VCC" H 7550 4300 50  0000 C CNN
+F 2 "" H 7550 4150 50  0000 C CNN
+F 3 "" H 7550 4150 50  0000 C CNN
+	1    7550 4150
+	1    0    0    -1
+$EndComp
+Wire Wire Line
+	7550 4150 7550 4250
+Wire Wire Line
+	8050 5000 8000 5000
+Text HLabel 8400 4600 2    60   Input ~ 0
+CTRL_EXT1
+Wire Wire Line
+	8400 4600 8300 4600
 $EndSCHEMATC
